Commit message: Updated Image - humble full - fixed display - added claude - gazebo binaries - gzros2control source

File: src/simple_robot/urdf/simple_robot.urdf (robot description, URDF)
Before this commit: robot simple_robot, 6 links, 5 joints
Joints:
- joint front_left_wheel_joint: limit (none) -> effort=10 velocity=10
- joint front_right_wheel_joint: limit (none) -> effort=10 velocity=10
